Commit message: Zmiany na potrzebyintegracji z ros melodic (zamiana boosta na c++11)

File: yumi_description/urdf/yumi.urdf.xacro (robot description, xacro)
@@ -11,4 +11,13 @@
   <!-- Import Gazebo plugins -->
   <xacro:include filename="$(find yumi_description)/urdf/Gazebo/gazebo.urdf.xacro"/>
+  <xacro:if value="${yumi_setup == 'default'}">
+    <xacro:property name="yumi_parent" value="world" />
+    <link name="world"/>
+    <joint name="world_joint" type="fixed">
+      <parent link="world"/>
+      <child link="yumi_base_link"/>
+      <origin xyz="0 0 0.1" rpy="0 0 0" />
+    </joint>
+  </xacro:if>
   <!--yumi-->
   <xacro:yumi name="yumi" hardware_interface="hardware_interface/$(arg arms_interface)" parent="${yumi_parent}" >
@@ -27,12 +36,3 @@
   	<!-- Pure YuMi URDF, with no joints connecting it to any other robot or pedestal. Neither accessories. -->
   </xacro:if>
-  <xacro:if value="${yumi_setup == 'default'}">
-    <xacro:property name="yumi_parent" value="world" />
-    <link name="world"/>
-    <joint name="world_joint" type="fixed">
-      <parent link="world"/>
-      <child link="yumi_base_link"/>
-      <origin xyz="0 0 0.1" rpy="0 0 0" />
-    </joint>
-  </xacro:if>
 </robot>

Commit message: Fix wrong placement of yumi setup

File: yumi_description/urdf/yumi.urdf.xacro (robot description, xacro)
@@ -11,4 +11,5 @@
   <!-- Import Gazebo plugins -->
   <xacro:include filename="$(find yumi_description)/urdf/Gazebo/gazebo.urdf.xacro"/>
+  <xacro:property name="yumi_setup" value="$(arg yumi_setup)" />
   <xacro:if value="${yumi_setup == 'default'}">
     <xacro:property name="yumi_parent" value="world" />
@@ -32,5 +33,4 @@
     <origin xyz="0 0 0.007" rpy="0 0 ${PI}" />
   </xacro:yumi_servo_gripper>
-  <xacro:property name="yumi_setup" value="$(arg yumi_setup)" />
   <xacro:if value="${yumi_setup == 'robot_centric'}">
   	<!-- Pure YuMi URDF, with no joints connecting it to any other robot or pedestal. Neither accessories. -->
